File: test/test.kicad_sch (KiCad schematic)
At the start: 0 parts

Commit message: said hi to alan
Other:
- note added: "Hi alan this is a test"
Changed lines of the file:
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@@
 	(generator_version "9.0")
 	(paper "A4")
+	(text "Hi alan this is a test"
+		(exclude_from_sim no)
+		(at 88.646 82.296 0)
+		(effects
+			(font
+				(size 1.27 1.27)
+			)
+		)
+	)
 	(symbol
 		(lib_id "power:+1V0")
