File: IndividualFolders/Landon Doughty/landons project/landons project.kicad_pcb (KiCad board)
At the start: 2 copper layers, 41.5 x 56.5 mm, 1 part

Commit message: landons changes
Parts:
- moved G*** 77.4 mm to (195.0, 71.5)
Other:
- board size 41.5 x 56.5 mm -> 76.2 x 76.2 mm
Changed lines of the file:
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@@
 	(footprint "logos:ECLIPSELogo1"
 		(layer "F.Cu")
-		(at 118 79.5)
+		(at 195 71.5)
 		(property "Reference" "G***"
 			(at -0.5 -6.5 0)
@@
 		(embedded_fonts no)
 	)
-	(gr_line
-		(start 97 127.5)
-		(end 97 77)
+	(gr_circle
+		(center 195 97.5)
+		(end 233.1 97.5)
 		(stroke
 			(width 0.05)
 			(type default)
 		)
+		(fill no)
 		(layer "Edge.Cuts")
 	)
-	(gr_arc
-		(start 135.5 74)
-		(mid 137.62132 74.87868)
-		(end 138.5 77)
+	(gr_circle
+		(center 195 97.5)
+		(end 207.7 97.5)
 		(stroke
 			(width 0.05)
 			(type default)
 		)
+		(fill no)
 		(layer "Edge.Cuts")
 	)
-	(gr_arc
-		(start 97 77)
-		(mid 97.87868 74.87868)
-		(end 100 74)
-		(stroke
-			(width 0.05)
-			(type default)
-		)
-		(layer "Edge.Cuts")
-	)
-	(gr_line
-		(start 100 74)
-		(end 135.5 74)
-		(stroke
-			(width 0.05)
-			(type default)
-		)
-		(layer "Edge.Cuts")
-	)
-	(gr_arc
-		(start 138.5 127.5)
-		(mid 137.62132 129.62132)
-		(end 135.5 130.5)
-		(stroke
-			(width 0.05)
-			(type default)
-		)
-		(layer "Edge.Cuts")
-	)
-	(gr_line
-		(start 138.5 77)
-		(end 138.5 127.5)
-		(stroke
-			(width 0.05)
-			(type default)
-		)
-		(layer "Edge.Cuts")
-	)
-	(gr_line
-		(start 135.5 130.5)
-		(end 100 130.5)
-		(stroke
-			(width 0.05)
-			(type default)
-		)
-		(layer "Edge.Cuts")
-	)
-	(gr_arc
-		(start 100 130.5)
-		(mid 97.87868 129.62132)
-		(end 97 127.5)
-		(stroke
-			(width 0.05)
-			(type default)
-		)
-		(layer "Edge.Cuts")
-	)
