File: IndividualFolders/Alan Bailey/Alans project/Alans project.kicad_sch (KiCad schematic)
At the start: 0 parts

Commit message: Made the recommended circuit for the MMC5983MA
Parts:
- added C1: 1u, symbol Device:C
- added C2: 10u, symbol Device:C
- added U1: MMC5983MA, MMC5983MA_MEM, symbol MMC5983MA:MMC5983MA
Connections:
- new net: C2.1, U1.10 (CAP)
- new net +3.3V: C1.1, U1.13 (VDDIO), U1.2 (VDD)
- new net GND: C1.2, C2.2, U1.11 (GND), U1.9 (GND)
- new net SCL/SPI_5CK: U1.1 (SCL/SPI_SCK)
- new net SDA/SPI_5DI: U1.16 (SDA/SPI_SDI)
- new net SPI_CS: U1.4 (SPI_CS)
- new net SPI_SD0: U1.5 (SPI_SDO)

Commit message: add footprint and make basic pcb
Parts:
- C1, C2: footprint (none) -> Capacitor_SMD:C_0805_2012Metric
- U1: footprint MMC5983MA_MEM -> Package_LGA:LGA-16_3x3mm_P0.5mm
Changed lines of the file:
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@@
 			)
 		)
-		(property "Footprint" ""
+		(property "Footprint" "Capacitor_SMD:C_0805_2012Metric"
 			(at 191.77 108.2548 0)
 			(effects
@@
 			)
 		)
-		(property "Footprint" ""
+		(property "Footprint" "Capacitor_SMD:C_0805_2012Metric"
 			(at 147.32 126.0348 0)
 			(effects
@@
 			)
 		)
-		(property "Footprint" "MMC5983MA_MEM"
+		(property "Footprint" "Package_LGA:LGA-16_3x3mm_P0.5mm"
 			(at 110.49 93.98 0)
 			(effects
