File: IndividualFolders/Reza Rahimzadeh/Reza's Project/KX134/KX134.kicad_sch (KiCad schematic)
At the start: 3 parts, among them U1 KX134-1211

Commit message: Updated KX134 Schematic
Connections:
- net ACCEL_IOVDD renamed IO_VDD
- net ACCEL_VDD renamed VDD

Commit message: Select footprint's and make basic PCB for KX134
Parts:
- C1, C2: footprint (none) -> Capacitor_SMD:C_0805_2012Metric
- U1: footprint LGA12_2X2X0P9_ROM -> Package_LGA:LGA-12_2x2mm_P0.5mm
Changed lines of the file:
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@@
 			)
 		)
-		(property "Footprint" ""
+		(property "Footprint" "Capacitor_SMD:C_0805_2012Metric"
 			(at 115.2652 111.76 0)
 			(effects
@@
 			)
 		)
-		(property "Footprint" ""
+		(property "Footprint" "Capacitor_SMD:C_0805_2012Metric"
 			(at 178.7652 105.41 0)
 			(effects
@@
 			)
 		)
-		(property "Footprint" "LGA12_2X2X0P9_ROM"
+		(property "Footprint" "Package_LGA:LGA-12_2x2mm_P0.5mm"
 			(at 115.57 90.17 0)
 			(effects
