File: IndividualFolders/Brian Dai/Switching Voltage Regulator/Switching Voltage Regulator.kicad_sch (KiCad schematic)
At the start: 5 parts, among them U1 LM2575-3.3BT

Commit message: Choose footprints for LM2575 power regulator. May need to be changed. HIGH POWER
Parts:
- C1, C2: footprint (none) -> Capacitor_SMD:C_0805_2012Metric
- D1: footprint (none) -> Diode_SMD:D_0805_2012Metric
- L1: footprint (none) -> Inductor_SMD:L_0805_2012Metric
- U1: footprint Package_TO_SOT_THT:TO-220-5_Vertical -> Package_TO_SOT_SMD:TO-263-5_TabPin3
Changed lines of the file:
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@@
 			)
 		)
-		(property "Footprint" ""
+		(property "Footprint" "Inductor_SMD:L_0805_2012Metric"
 			(at 170.18 97.79 0)
 			(effects
@@
 			)
 		)
-		(property "Footprint" ""
+		(property "Footprint" "Capacitor_SMD:C_0805_2012Metric"
 			(at 176.2252 106.68 0)
 			(effects
@@
 			)
 		)
-		(property "Footprint" ""
+		(property "Footprint" "Capacitor_SMD:C_0805_2012Metric"
 			(at 127.9652 97.79 0)
 			(effects
@@
 			)
 		)
-		(property "Footprint" "Package_TO_SOT_THT:TO-220-5_Vertical"
+		(property "Footprint" "Package_TO_SOT_SMD:TO-263-5_TabPin3"
 			(at 148.59 101.6 0)
 			(effects
@@
 			)
 		)
-		(property "Footprint" ""
+		(property "Footprint" "Diode_SMD:D_0805_2012Metric"
 			(at 165.1 102.87 0)
 			(effects
