File: IndividualFolders/Tyler/MCS1802 schematic/MCS1802 schematic.kicad_sch (KiCad schematic)
At the start: 3 parts, among them U1 MCS1802GS-50-Z

Commit message: mcs1802
Parts:
- removed Cf: C, symbol Device:C
- C1: value 0.1 uf -> 1 µf; footprint (none) -> Capacitor_SMD:C_0805_2012Metric
- U1: footprint SOIC-8_MNP -> Package_SO:SOIC-8_3.9x4.9mm_P1.27mm
Connections:
- no-connect marks 0 -> 1
Changed lines of the file:
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@@
 		(color 0 0 0 0)
 	)
-	(junction
-		(at 144.78 86.36)
-		(diameter 0)
-		(color 0 0 0 0)
+	(no_connect
+		(at 137.16 76.2)
 	)
 	(wire
@@
 	(wire
 		(pts
-			(xy 144.78 83.82) (xy 144.78 86.36)
-		)
-		(stroke
-			(width 0)
-			(type default)
-		)
-	)
-	(wire
-		(pts
 			(xy 86.36 78.74) (xy 96.52 78.74)
 		)
@@
 		(pts
 			(xy 96.52 71.12) (xy 96.52 73.66)
-		)
-		(stroke
-			(width 0)
-			(type default)
-		)
-	)
-	(wire
-		(pts
-			(xy 137.16 76.2) (xy 144.78 76.2)
 		)
 		(stroke
@@
 				(justify right)
 				(hide yes)
-			)
-		)
-	)
-	(symbol
-		(lib_id "Device:C")
-		(at 144.78 80.01 0)
-		(unit 1)
-		(exclude_from_sim no)
-		(in_bom yes)
-		(on_board yes)
-		(dnp no)
-		(fields_autoplaced yes)
-		(property "Reference" "Cf"
-			(at 148.59 78.7399 0)
-			(effects
-				(font
-					(size 1.27 1.27)
-				)
-				(justify left)
-			)
-		)
-		(property "Value" "C"
-			(at 148.59 81.2799 0)
-			(effects
-				(font
-					(size 1.27 1.27)
-				)
-				(justify left)
-			)
-		)
-		(property "Footprint" ""
-			(at 145.7452 83.82 0)
-			(effects
-				(font
-					(size 1.27 1.27)
-				)
-				(hide yes)
-			)
-		)
-		(property "Datasheet" "~"
-			(at 144.78 80.01 0)
-			(effects
-				(font
-					(size 1.27 1.27)
-				)
-				(hide yes)
-			)
-		)
-		(property "Description" "Unpolarized capacitor"
-			(at 144.78 80.01 0)
-			(effects
-				(font
-					(size 1.27 1.27)
-				)
-				(hide yes)
-			)
-		)
-		(pin "2"
-		)
-		(pin "1"
-		)
-		(instances
-			(project ""
-				(path "/7c0919ff-f8bd-446a-9f9b-2fa64e9478a1"
-					(reference "Cf")
-					(unit 1)
-				)
 			)
 		)
@@
 			)
 		)
-		(property "Value" "0.1 uf"
+		(property "Value" "1 µf"
 			(at 165.1 76.1999 0)
 			(effects
@@
 			)
 		)
-		(property "Footprint" ""
+		(property "Footprint" "Capacitor_SMD:C_0805_2012Metric"
 			(at 162.2552 78.74 0)
 			(effects
@@
 			)
 		)
-		(property "Footprint" "SOIC-8_MNP"
+		(property "Footprint" "Package_SO:SOIC-8_3.9x4.9mm_P1.27mm"
 			(at 96.52 71.12 0)
 			(effects
