File: IndividualFolders/Brian Dai/Main1/Main.kicad_sch (KiCad schematic)
At the start: 96 parts, among them J1 USB_B_Micro, J2 XT60, J3 Conn_01x03, J4 Conn_01x03, J5 Conn_01x03, J6 Conn_01x03, J7 MSD-4-A, J9 Conn_01x03, Q2 Si2301CDS, SW1 SW_Push, SW2 SW_Push, U1 RP2350A-QFN60, U10 LM75B, U11 MCS1802GS-50-Z, U12 MCS1802GS-50-Z, U13 MCS1802GS-50-Z, U15 AP62150WU, U2 W25Q128JVS, U3 AMS1117-3.3, U4 MMC5983MA, U5 ICM-42688-P, U6 INA226, U7 KX134-1211, U8 MS5611-01BA, U9 MCS1802GS-50-Z, Y1 ABM8-272-T3

Commit message: Meeting 2/28/26
Parts:
- removed C37, C39: 10u, Capacitor_SMD:C_0805_2012Metric, symbol Device:C
- removed C38, C40: 100n, Capacitor_SMD:C_0402_1005Metric, symbol Device:C
- removed C41: 22u, Capacitor_SMD:C_0805_2012Metric, symbol Device:C
- removed J2: XT60, Connector_AMASS:AMASS_XT60-M_1x02_P7.20mm_Vertical, symbol Connector_Generic:Conn_01x02
- removed J7: MSD-4-A, otherComponents:CUI_MSD-4-A, symbol otherSymbols:MSD-4-A
- removed J9: Conn_01x03, Connector_PinHeader_2.54mm:PinHeader_1x03_P2.54mm_Vertical, symbol Connector_Generic:Conn_01x03
- removed L3: 3.3u, Inductor_SMD:L_1008_2520Metric_Pad1.43x2.20mm_HandSolder, symbol Device:L
- removed Q2: Si2301CDS, Package_TO_SOT_SMD:SOT-23, symbol Transistor_FET:Si2319CDS
- removed R14, R15, R16, R17, R18, R21, R9: 10k, Resistor_SMD:R_0402_1005Metric, symbol Device:R
- removed R20: 30k, Resistor_SMD:R_0603_1608Metric, symbol Device:R
- removed R22: 100k, Resistor_SMD:R_0402_1005Metric, symbol Device:R
- removed R23: 1k, Resistor_SMD:R_0402_1005Metric, symbol Device:R
- removed U15: AP62150WU, Package_TO_SOT_SMD:TSOT-23-6, symbol Regulator_Switching:AP62150WU
- added C35: 100uF, symbol Device:C
- added C36: 330uF, symbol Device:C
- added D4: 1N5189, symbol Device:D
- added J2: Micro_SD_Card, symbol Connector:Micro_SD_Card
- added L2: 330uH, symbol Device:L
- added U14: LM2575-3.3BT, Package_TO_SOT_SMD:TO-263-5_TabPin3, symbol Regulator_Switching:LM2575-3.3BT
- D1: value RED_LED -> LED
- D2: value BLUE_LED -> LED
- D3: value GREEN_LED -> LED
Connections:
- net GND: now also R13.1, U6.8 (Vbus), U6.9 (Vin-), C35.2, C36.2, D4.2 (A), U14.3 (GND), U14.5 (~{ON}/OFF); no longer C29.2, C30.2
- net SCL: no longer U1.33 (GPIO21)
- net SDA: no longer U1.32 (GPIO20)
- net SPI_SD0: no longer U7.1 (SDO/ADDR)
- net SPI_SDI: no longer U7.2 (SDI/SDA)
- net VIN: now also C35.1, U14.1 (VIN); no longer R13.1, U11.1 (IP+), U11.2 (IP+), U12.3 (IP-), U12.4 (IP-), U13.1 (IP+), U13.2 (IP+), U6.9 (Vin-), U9.3 (IP-), U9.4 (IP-)
- net Vout1: no longer U1.40 (GPIO26_ADC0)
- net Vout2: no longer U1.41 (GPIO27_ADC1)
- net Vout3: no longer U1.43 (GPIO29_ADC3)
- net Vout4: no longer U1.42 (GPIO28_ADC2)
- net VSS: now reaches R13.2, U6.10 (Vin+)
- net VSS: no longer U6.8 (Vbus)
- new net: D4.1 (K), L2.1, U14.2 (OUT)
- new net: C29.2, C30.2
- new net ACCEL_SDI/SDA: U7.2 (SDI/SDA)
- new net ACCEL_SDO/ADDR: U7.1 (SDO/ADDR)
- new net VOUT: C36.1, L2.2, U14.4 (FB)
- new net current +: U11.1 (IP+), U11.2 (IP+), U12.3 (IP-), U12.4 (IP-), U13.1 (IP+), U13.2 (IP+), U9.3 (IP-), U9.4 (IP-)
- no-connect marks 10 -> 9
Other:
- note removed: "Blocks Connection when USB plugged in to prevent backpowering"
- moved on the sheet: C24, D1, D2, D3, R10, R11, R12, R13, R7, R8, U6
