File: IndividualFolders/Michael Chekler/Main.kicad_pcb (KiCad board)
At the start: 4 copper layers, 76.2 x 64.9 mm, 79 parts, among them J1 USB_B_Micro, J2 Conn_01x02, J3 Conn_01x03, J4 Conn_01x03, J5 Conn_01x03, J6 Conn_01x03, J7 MSD-4-A, SW1 SW_Push, SW2 SW_Push, U1 RP2350A-QFN60, U10 LM75B, U11 MCS1802GS-50-Z, U12 MCS1802GS-50-Z, U13 MCS1802GS-50-Z, U14 LM2575-3.3BT, U2 W25Q128JVS, U3 AMS1117-3.3, U4 MMC5983MA, U5 ICM-42688-P, U6 INA226, U7 KX134-1211, U8 MS5611-01BA, U9 MCS1802GS-50-Z, Y1 ABM8-272-T3

Commit message: Main PCB practice wiring
Parts:
- moved C18 101.7 mm to (82.5, 119.0), turned to 180 degrees
- moved C11 100.3 mm to (68.0, 119.5), turned to 90 degrees
- moved C12 98.4 mm to (70.0, 119.5), turned to 90 degrees
- moved C13 97.1 mm to (73.0, 119.5), turned to 90 degrees
- moved C19 96.6 mm to (82.5, 116.0), turned to 180 degrees
- moved C14 95.9 mm to (76.0, 119.5), turned to 90 degrees
- moved C15 95.0 mm to (79.0, 119.5), turned to 90 degrees
- moved U14 94.2 mm to (120.2, 104.1), turned to 90 degrees
- moved C23 92.8 mm to (86.0, 106.0)
- moved C20 91.6 mm to (82.5, 113.0), turned to 180 degrees
- moved R7 88.9 mm to (81.0, 116.5), turned to 90 degrees
- moved C21 86.6 mm to (82.5, 110.0), turned to 180 degrees
- moved C25 85.0 mm to (81.0, 106.0)
- moved J3 84.8 mm to (90.9, 87.0), turned to 90 degrees
- moved J2 84.0 mm to (114.0, 129.6), turned to 90 degrees
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