File: IndividualFolders/Tyler/Main/Main.kicad_sch (KiCad schematic)
At the start: 82 parts, among them J1 USB_B_Micro, J2 Conn_01x02, J3 Conn_01x03, J4 Conn_01x03, J5 Conn_01x03, J6 Conn_01x03, J7 MSD-4-A, SW1 SW_Push, SW2 SW_Push, U1 RP2350A-QFN60, U10 LM75B, U11 MCS1802GS-50-Z, U12 MCS1802GS-50-Z, U13 MCS1802GS-50-Z, U14 LM2575-3.3BT, U2 W25Q128JVS, U3 AMS1117-3.3, U4 MMC5983MA, U5 ICM-42688-P, U6 INA226, U7 KX134-1211, U8 MS5611-01BA, U9 MCS1802GS-50-Z, Y1 ABM8-272-T3

Commit message: idk man
Parts:
- removed C35: 100uF, symbol Device:C
- removed C36: 330uF, symbol Device:C
- removed D4: 1N5189, symbol Device:D
- removed L2: 330uH, symbol Device:L
- removed U14: LM2575-3.3BT, Package_TO_SOT_SMD:TO-263-5_TabPin3, symbol Regulator_Switching:LM2575-3.3BT
- added C37, C39: 10u, Capacitor_SMD:C_0805_2012Metric, symbol Device:C
- added C38, C40: 100n, Capacitor_SMD:C_0402_1005Metric, symbol Device:C
- added C41: 22u, Capacitor_SMD:C_0805_2012Metric, symbol Device:C
- added J9: Conn_01x03, Connector_PinHeader_2.54mm:PinHeader_1x03_P2.54mm_Vertical, symbol Connector_Generic:Conn_01x03
- added L3: 3.3u, Inductor_SMD:L_1008_2520Metric_Pad1.43x2.20mm_HandSolder, symbol Device:L
- added Q2: Si2301CDS, Package_TO_SOT_SMD:SOT-23, symbol Transistor_FET:Si2319CDS
- added R14, R15, R16, R17, R18, R21, R9: 10k, Resistor_SMD:R_0402_1005Metric, symbol Device:R
- added R20: 30k, Resistor_SMD:R_0603_1608Metric, symbol Device:R
- added R22: 100k, Resistor_SMD:R_0402_1005Metric, symbol Device:R
- added R23: 1k, Resistor_SMD:R_0402_1005Metric, symbol Device:R
- added U15: AP62150WU, Package_TO_SOT_SMD:TSOT-23-6, symbol Regulator_Switching:AP62150WU
- D1: value LED -> RED_LED
- D2: value LED -> BLUE_LED
- D3: value LED -> GREEN_LED
- J2: value Conn_01x02 -> XT60
Connections:
- net ACCEL_SDI/SDA is gone; now on net SPI_SDI: U7.2 (SDI/SDA)
- net ACCEL_SDO/ADDR is gone; now on net SPI_SD0: U7.1 (SDO/ADDR)
- net current + is gone; now on net VIN: U12.3 (IP-), U12.4 (IP-), U9.3 (IP-), U9.4 (IP-)
- net +3.3V: now also J7.4 (VDD), C37.1, C38.1, Q2.3 (D), R14.2, R15.1, R16.1, R17.1, R18.1, R9.2
- net ACCEL_nCS: now also U1.17 (GPIO13)
- net GND: now also C29.2, C30.2, J7.6 (VSS), J7.G1 (COVER_GND), J7.G2 (COVER_GND__1), J7.G3 (COVER_GND__2), J7.G4 (COVER_GND__3), C37.2, C38.2, C39.2, C41.2, J9.1 (Pin_1), R21.2, R22.1, U15.1 (GND); no longer R13.1, U6.8 (Vbus), U6.9 (Vin-)
- net ICM_CS: now also U1.13 (GPIO9)
- net MMC_CS: now also U1.28 (GPIO17)
- net SCL: now also U1.33 (GPIO21)
- net SDA: now also U1.32 (GPIO20)
- net SPI_SCK: now also U1.14 (GPIO10)
- net SPI_SD0: now also U1.16 (GPIO12)
- net SPI_SDI: now also U1.15 (GPIO11)
- net VBUS: now also Q2.1 (G), R22.2
- net VIN: now also R13.1, U6.9 (Vin-), C39.1, U15.3 (VIN); no longer J2.2 (Pin_2), U12.1 (IP+), U12.2 (IP+), U9.1 (IP+), U9.2 (IP+)
- net Vout1: now also U1.40 (GPIO26_ADC0)
- net Vout2: now also U1.41 (GPIO27_ADC1)
- net Vout3: now also U1.43 (GPIO29_ADC3)
- net Vout4: now also U1.42 (GPIO28_ADC2)
- net current -2: now also U9.1 (IP+), U9.2 (IP+)
- net current -3: now also U12.1 (IP+), U12.2 (IP+)
- net at J7.1 (DAT2): now also R14.1
- net SD_ChipSelect: now reaches J7.2 (CD/DAT3)
- net SPI_SDI2: now reaches J7.3 (CMD)
- net SPI_SDI2: now also R17.2
- net SPI_SCLK2: now reaches J7.5 (CLK)
- net SPI_SCLK2: now also R18.2
- net SPI_SDO2: now reaches J7.7 (DAT0)
- net SPI_SDO2: now also R16.2
- net at J7.8 (DAT1): now also R9.1
- net SD_CD: now reaches J7.CD
- net SD_CD: now also R15.2
- net at U1.24 (SWCLK): now also J9.3 (Pin_3)
- net at U1.25 (SWDIO): now also J9.2 (Pin_2)
- net VSS: no longer names the net of R13.2, U6.10 (Vin+)
- net VSS: now also J2.2 (Pin_2), U6.8 (Vbus)
- new net: C41.1, L3.1, Q2.2 (S), R20.1
- new net: C40.1, L3.2, U15.2 (SW)
- new net: C40.2, U15.6 (BST)
- new net: R20.2, R23.1
- new net: R21.1, R23.2, U15.4 (FB)
- no-connect marks 9 -> 10
Other:
- note added: "Blocks Connection when USB plugged in to prevent backpowering"
- note removed: "figure out connection of 3.3v sources"
- moved on the sheet: C24, D1, D2, D3, J2, R10, R11, R12, R13, R7, R8, U6
