File: IndividualFolders/Brian Dai/Main/Main.kicad_sch (KiCad schematic)
At the start: 96 parts, among them J1 USB_B_Micro, J2 XT60, J3 Conn_01x03, J4 Conn_01x03, J5 Conn_01x03, J6 Conn_01x03, J7 MSD-4-A, J9 Conn_01x03, Q2 Si2301CDS, SW1 SW_Push, SW2 SW_Push, U1 RP2350A-QFN60, U10 LM75B, U11 MCS1802GS-50-Z, U12 MCS1802GS-50-Z, U13 MCS1802GS-50-Z, U15 AP62150WU, U2 W25Q128JVS, U3 AMS1117-3.3, U4 MMC5983MA, U5 ICM-42688-P, U6 INA226, U7 KX134-1211, U8 MS5611-01BA, U9 MCS1802GS-50-Z, Y1 ABM8-272-T3

Commit message: Resistor component numbers
Parts:
- removed Q2: Si2301CDS, Package_TO_SOT_SMD:SOT-23, symbol Transistor_FET:Si2319CDS
- added C35: 1u, Capacitor_SMD:C_0805_2012Metric, symbol Device:C_Small
- added D4: RED_LED, LED_SMD:LED_0805_2012Metric, symbol Device:LED
- added R19: 30k, Resistor_SMD:R_0402_1005Metric, symbol Device:R_Small_US
- added R24, R25, R26, R27: 100k, Resistor_SMD:R_0402_1005Metric, symbol Device:R_Small_US
- added U14: TPS2121RUXR, Package_DFN_QFN:Texas_VQFN-HR-12_2x2.5mm_P0.5mm, symbol TPS2121RUXR:TPS2121RUXR
- D2: value BLUE_LED -> YELLOW_LED
- R10: value R -> 60
- R20: footprint Resistor_SMD:R_0603_1608Metric -> Resistor_SMD:R_0402_1005Metric
- R22: value 100k -> 60
Connections:
- net ACCEL_INT1 is gone; now on net ACCEL_INT: U7.5 (INT1)
- net ACCEL_nCS is gone; now on net ACCEL_CS: U7.10 (nCS)
- net IO_VDD is gone; now on net +3.3V: C25.1, U7.3 (IO_VDD)
- net SCLK is gone; now on net SPI_SCK: U8.8 (SCLK)
- net SDI is gone; now on net SPI_SDI: U8.7 (SDI/SDA)
- net SDO is gone; now on net SPI_SDO: U8.6 (SDO)
- net SPI_SD0 is gone; now on net SPI_SDO: U4.5 (SPI_SDO), U5.1 (AP_SDO/AP_AD0), U7.1 (SDO/ADDR)
- net VDD is gone; now on net +3.3V: C26.2, U7.7 (VDD)
- net +3.3V: now also R22.1, U14.1 (OUT), U14.8 (OUT); no longer C21.1, U3.2 (VO)
- net GND: now also C35.2, R24.2, R26.2, R27.2, U14.12 (GND), U14.4 (OV2), U14.5 (OV1); no longer R22.1
- net ICM_CS: now also U1.17 (GPIO13)
- net INT2/DRDY: now also U1.27 (GPIO16)
- net MMC_CS: now also U1.18 (GPIO14)
- net MS5611_CS: now also U1.16 (GPIO12)
- net PWM1: now also U1.31 (GPIO19)
- net PWM2: now also U1.34 (GPIO22)
- net PWM3: now also U1.36 (GPIO24)
- net PWM4: now also U1.35 (GPIO23)
- net SD_CD: now also U1.7 (GPIO4)
- net SD_ChipSelect: now also U1.3 (GPIO1)
- net SPI_SCK: now also U1.14 (GPIO10)
- net SPI_SCLK2: now also U1.4 (GPIO2)
- net SPI_SDI: now also U1.15 (GPIO11)
- net SPI_SDI2: now also U1.5 (GPIO3)
- net SPI_SDO2: now also U1.2 (GPIO0)
- net VBUS: no longer R22.2
- net 3.3v_Batt: now reaches C41.1, L3.1, R20.1
- net 3.3v_Batt: now also R25.1, U14.2 (IN2)
- net MMC_INT: now reaches U4.15 (INT)
- net MMC_INT: now also U1.29 (GPIO18)
- net SPI_SDO: now reaches U1.12 (GPIO8)
- net ACCEL_CS: now reaches U1.19 (GPIO15)
- net ACCEL_INT: now reaches U1.28 (GPIO17)
- net ACCEL_INT2: no longer names the net of U7.6 (INT2)
- new net: R25.2, R26.1, U14.3 (CP2)
- new net: R19.2, R24.1, U14.6 (PR1)
- new net: D4.1 (K), U14.9 (ST)
- new net: D4.2 (A), R22.2
- new net: R27.1, U14.10 (ILIM)
- new net: C35.1, U14.11 (SS)
- new net 3.3v_usb: C21.1, R19.1, U14.7 (IN1), U3.2 (VO)
Other:
- note added: "INT HIGH when reading available"
- note added: "SPI_1: ICM (IMU) KX-134(HIGH G-Accel) MMC (Magnetometer) MS5611 (Barometer)"
- note removed: "Blocks Connection when USB plugged in to prevent backpowering"
- moved on the sheet: U8
