File: Version2/Version2.kicad_pcb (KiCad board)
At the start: 4 copper layers, 50.8 x 106.6 mm, 136 parts, among them J1 USB_C_Receptacle_USB2.0_16P, J10 Conn_01x03, J11 Conn_01x03, J12 MSD-4-A, J13 Conn_01x04_Socket, J14 Conn_01x03, J15 Conn_01x03, J16 Conn_01x03, J17 Conn_01x03, J18 Conn_01x04_Socket, J19 Conn_01x04_Socket, J20 Screw_Terminal_01x02, J21 Screw_Terminal_01x02, J26 Conn_01x04_Socket, J27 Conn_01x02_Socket, J29 Conn_01x02_Socket, J30 Conn_01x02_Socket, J31 Conn_01x02_Socket, J4 Screw_Terminal_01x02, J5 Conn_01x02_Pin, J6 Conn_01x04_Socket, J7 Conn_01x03, J8 Conn_01x03, J9 Conn_01x04_Socket, SW1 SW_Push, SW2 SW_Push, U1 W25Q128JVS, U10 INA219AxDCN, U11 AP2112K-3.3, U12 AP62150WU, U13 TPS2121RUXR, U14 AP62150WU, U15 74AHC541, U2 RP2350B-QFN80, U3 MMC5983MA, U4 ICM-45686, U5 MS5611-01BA, U6 TMP117xxDRV, U8 KX134-1211, U9 TPS2121RUXR, Y1 ABM8-272-T3

Commit message: Manufacturable but Needs Thorough Check Through
Parts:
- removed J20, J21, J4: Screw_Terminal_01x02, PCM_SparkFun-Connector:ScrewTerminal_1x02_P3.5mm_Horizontal_Black
- added G***: LOGO, logos:ECLIPSELogo1, F.Cu at (148.5, 78.0)
- moved J30 97.1 mm to (123.4, 138.4), turned to 90 degrees
- moved J31 96.1 mm to (170.6, 136.4), turned to -90 degrees
- moved J27 78.8 mm to (170.6, 130.1)
- moved J29 78.8 mm to (123.4, 132.1)
- moved J6 62.2 mm to (170.6, 119.8)
- moved J9 41.6 mm to (123.4, 125.8)
- moved H1 33.7 mm to (169.4, 75.8)
- moved H2 33.7 mm to (124.6, 75.8)
- moved J26 24.4 mm to (123.4, 87.9)
- moved J18 24.4 mm to (123.4, 98.2)
- moved J12 14.3 mm to (131.5, 109.0)
- moved C46 14.3 mm to (165.8, 154.0)
- moved C47 14.3 mm to (154.6, 154.0)
- moved G2 14.3 mm to (160.2, 155.3)
- moved H4 14.3 mm to (169.4, 156.8)
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Connections:
- J26 pad 2: GPIO1 -> XTRA_SPI_CS
- U2 pad 11: unconnected-(U2-GPIO12-Pad11) -> UART0_TX
- U2 pad 12: unconnected-(U2-GPIO13-Pad12) -> UART0_RX
- U2 pad 28: unconnected-(U2-GPIO27-Pad28) -> XTRA_SPI_CS
- U2 pad 36: unconnected-(U2-GPIO28-Pad36) -> SPI_MISO_SD
- U2 pad 37: unconnected-(U2-GPIO29-Pad37) -> SD_ChipSelect
- U2 pad 38: unconnected-(U2-GPIO30-Pad38) -> SPI_SCK_SD
- U2 pad 39: unconnected-(U2-GPIO31-Pad39) -> SPI_MOSI_SD
- U2 pad 45: SPI_MISO_SD -> unconnected-(U2-GPIO36-Pad45)
- U2 pad 46: SD_ChipSelect -> unconnected-(U2-GPIO37-Pad46)
- U2 pad 47: SPI_SCK_SD -> unconnected-(U2-GPIO38-Pad47)
- U2 pad 48: SPI_MOSI_SD -> unconnected-(U2-GPIO39-Pad48)
- U2 pad 77: unconnected-(U2-GPIO0-Pad77) -> GPIO0
- U2 pad 78: unconnected-(U2-GPIO1-Pad78) -> GPIO1
- U2 pad 79: unconnected-(U2-GPIO2-Pad79) -> GPIO2
- U2 pad 8: unconnected-(U2-GPIO10-Pad8) -> SDA2
- U2 pad 80: unconnected-(U2-GPIO3-Pad80) -> GPIO3
- U2 pad 9: unconnected-(U2-GPIO11-Pad9) -> SCL2
Routing:
- net GPIO1: track 96.6 -> 41.3 mm, vias 3 -> 1
- net +5V: track 53.3 -> 5.75 mm
- net unconnected-(U2-GPIO42_ADC2-Pad53): track 32.7 -> 0.00 mm, vias 2 -> 0
- net XTRA_SPI_CS: track 0.00 -> 29.0 mm, vias 0 -> 2
- net +5V_USB: track 46.4 -> 20.4 mm, vias 10 -> 11
- net +3.3V: track 178.7 -> 152.9 mm, vias 47 -> 41
- net unconnected-(U2-GPIO43_ADC3-Pad54): track 24.4 -> 0.00 mm, vias 1 -> 0
- net unconnected-(U2-GPIO41_ADC1-Pad52): track 23.4 -> 0.00 mm, vias 2 -> 0
- net unconnected-(U2-GPIO40_ADC0-Pad49): track 20.3 -> 0.00 mm, vias 2 -> 0
- net unconnected-(U2-GPIO14-Pad13): track 14.3 -> 0.00 mm, vias 1 -> 0
- net GPIO3: track 47.9 -> 35.0 mm
- net SPI_MOSI_SEN: track 74.9 -> 64.9 mm, vias 1 -> 0
- net GPIO2: track 47.8 -> 38.4 mm
- net SPI_SCK_SEN: track 66.8 -> 59.5 mm
- net SWDIO: track 36.4 -> 29.7 mm
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- added copper zone on F.Cu, net +5V
- added copper zone on In2.Cu, net +5V
- added copper zone on In2.Cu, net +5V_USB
- added copper zone on In2.Cu, net 5v_Batt
- added copper zone on F.Cu, net GND
- added copper zone on In2.Cu, net GND
- added copper zone on In2.Cu, net VSYS
- removed copper zone on In1.Cu, net +5V_USB
- removed copper zone on In1.Cu, net 5v_Batt
Other:
- board size 50.8 x 106.6 mm -> 50.8 x 87 mm
- board text removed: "Batt 3V3"
- board text removed: "Batt 5V"
- board text removed: "D0"
- board text removed: "DO"
- board text removed: "SRC 3V3"
- board text removed: "SRC 5V"
- board text removed: "USB 3V3"
- board text removed: "USB 5V"
- board text removed: "VSYS"

Commit message: Small Fixes
Routing:
- net PWM7: track 12.9 -> 9.90 mm
- removed copper zone on In2.Cu, net +5V

Commit message: Added Test Points + Back Graphics
Parts:
- added C50: 10u, Capacitor_SMD:C_0805_2012Metric, B.Cu at (137.8, 125.4)
- added C51: 100n, Capacitor_SMD:C_0603_1608Metric, F.Cu at (151.4, 127.8)
- added G***: LOGO, logos:ECLIPSELogo1, B.Cu at (144.3, 77.9)
- added TP10: TestPoint_Small, TestPoint:TestPoint_Pad_1.0x1.0mm, B.Cu at (147.0, 96.1)
- added TP11: TestPoint_Small, TestPoint:TestPoint_Pad_1.0x1.0mm, B.Cu at (161.0, 126.4)
- added TP12: TestPoint_Small, TestPoint:TestPoint_Pad_1.0x1.0mm, B.Cu at (145.3, 125.7)
- added TP13: TestPoint_Small, TestPoint:TestPoint_Pad_1.0x1.0mm, B.Cu at (153.0, 131.6)
- added TP14: TestPoint_Small, TestPoint:TestPoint_Pad_1.0x1.0mm, B.Cu at (145.1, 131.8)
- added TP4: TestPoint_Small, TestPoint:TestPoint_Pad_1.0x1.0mm, B.Cu at (153.5, 91.7)
- added TP5: TestPoint_Small, TestPoint:TestPoint_Pad_1.0x1.0mm, B.Cu at (155.2, 87.8)
- added TP6: TestPoint_Small, TestPoint:TestPoint_Pad_1.0x1.0mm, B.Cu at (142.6, 90.6)
- added TP7: TestPoint_Small, TestPoint:TestPoint_Pad_1.0x1.0mm, B.Cu at (141.2, 90.6)
- added TP8: TestPoint_Small, TestPoint:TestPoint_Pad_1.0x1.0mm, B.Cu at (141.2, 98.0)
- added TP9: TestPoint_Small, TestPoint:TestPoint_Pad_1.0x1.0mm, B.Cu at (139.7, 98.0)
- U15: value 74AHC541 -> 74AHCT541
Routing:
- net GND: track 120.0 -> 127.2 mm
- net MAG_CS: track 17.8 -> 22.7 mm, vias 2 -> 3
- net Net-(U14-FB): track 0.00 -> 3.90 mm
- net Net-(U12-FB): track 0.00 -> 3.90 mm
- net BAR_CS: track 11.6 -> 13.5 mm, vias 0 -> 1
- net ACC_CS: track 11.6 -> 13.1 mm, vias 0 -> 1
- net +5V_USB: track 20.4 -> 21.6 mm
- removed copper zone on B.Cu, net Net-(U12-FB)
- removed copper zone on B.Cu, net Net-(U14-FB)
Other:
- board text added: "3.3 BATT"
- board text added: "3.3 USB"
- board text added: "5 BATT"
- board text added: "5 USB"
