File: Version2/Version2.kicad_sch (KiCad schematic)
At the start: 136 parts, among them J1 USB_C_Receptacle_USB2.0_16P, J10 Conn_01x03, J11 Conn_01x03, J12 MSD-4-A, J13 Conn_01x04_Socket, J14 Conn_01x03, J15 Conn_01x03, J16 Conn_01x03, J17 Conn_01x03, J18 Conn_01x04_Socket, J19 Conn_01x04_Socket, J20 Screw_Terminal_01x02, J21 Screw_Terminal_01x02, J24 Conn_01x04_Socket, J26 Conn_01x04_Socket, J27 Conn_01x02_Socket, J28 Conn_01x04_Socket, J29 Conn_01x02_Socket, J3 Screw_Terminal_01x02, J30 Conn_01x02_Socket, J31 Conn_01x02_Socket, J4 Screw_Terminal_01x02, J5 Conn_01x02_Pin, J6 Conn_01x04_Socket, J7 Conn_01x03, J8 Conn_01x03, J9 Conn_01x04_Socket, SW1 SW_Push, SW2 SW_Push, U1 W25Q128JVS, U10 INA219AxDCN, U11 AP2112K-3.3, U12 AP62150WU, U13 TPS2121RUXR, U14 AP62150WU, U15 74AHC541, U2 RP2350B-QFN80, U3 MMC5983MA, U4 ICM-45686, U5 MS5611-01BA, U6 TMP117xxDRV, U8 KX134-1211, U9 TPS2121RUXR, Y1 ABM8-272-T3

Commit message: Manufacturable but Needs Thorough Check Through
Parts:
- removed J20, J21, J3, J4: Screw_Terminal_01x02, PCM_SparkFun-Connector:ScrewTerminal_1x02_P3.5mm_Horizontal_Black, symbol Connector:Screw_Terminal_01x02
- removed J24, J28: Conn_01x04_Socket, Connector_JST:JST_PH_B4B-PH-K_1x04_P2.00mm_Vertical, symbol Connector:Conn_01x04_Socket
Connections:
- net GPIO0: now also U2.77 (GPIO0)
- net GPIO1: now also U2.78 (GPIO1); no longer J26.2 (Pin_2)
- net GPIO2: now also U2.79 (GPIO2)
- net GPIO3: now also U2.80 (GPIO3)
- net SCL2: now also U2.9 (GPIO11)
- net SDA2: now also U2.8 (GPIO10)
- net SD_ChipSelect: now also U2.37 (GPIO29); no longer U2.46 (GPIO37)
- net SPI_MISO_SD: now also U2.36 (GPIO28); no longer U2.45 (GPIO36)
- net SPI_MOSI_SD: now also U2.39 (GPIO31); no longer U2.48 (GPIO39)
- net SPI_SCK_SD: now also U2.38 (GPIO30); no longer U2.47 (GPIO38)
- net UART0_RX: now also U2.12 (GPIO13)
- net UART0_TX: now also U2.11 (GPIO12)
- net XTRA_SPI_CS: now reaches U2.28 (GPIO27)
- net XTRA_SPI_CS: now also J26.2 (Pin_2)
Other:
- note removed: "Secondary Radio connector"
- note removed: "V_OUT"
- note removed: "arm switch"
- moved on the sheet: J27, J29, J30, J31, J5

Commit message: Made Schematic more presentable
Connections:
- no-connect marks 12 -> 26
Other:
- note added: "Power Regulation"
- note added: "Power Switching"
- note added: "Sensors"
- moved on the sheet: C30, C31, C32, C33, C34, C35, C36, C37, C38, C39, C40, C41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

Commit message: Added Test Points + Back Graphics
Parts:
- added C50: 10u, Capacitor_SMD:C_0805_2012Metric, symbol Device:C
- added C51: 100n, Capacitor_SMD:C_0603_1608Metric, symbol Device:C
- added TP10, TP11, TP12, TP13, TP14, TP4, TP5, TP6, TP7, TP8, TP9: TestPoint_Small, TestPoint:TestPoint_Pad_1.0x1.0mm, symbol Connector:TestPoint_Small
- U15: value 74AHC541 -> 74AHCT541
Connections:
- net +5V: now also C50.1, C51.1
- net +5V_USB: now also TP12.1
- net 3.3v_Batt: now also TP13.1
- net 3.3v_usb: now also TP11.1
- net 5v_Batt: now also TP14.1
- net ACC_CS: now also TP8.1
- net ACC_INT: now also TP9.1
- net BAR_CS: now also TP10.1
- net GND: now also C50.2, C51.2
- net IMU_CS: now also TP5.1
- net IMU_INT1: now also TP4.1
- net MAG_CS: now also TP6.1
- net MAG_INT: now also TP7.1

Commit message: Updated LCSC Part Numbers
Parts:
- C1, C10, C11, C12, C17, C2, C21, C23, C24, C25, C28, C29, C30, C34, C38, C4, C41, C5, C51, C6, C7, C8, C9: LCSC Part Number C1525 -> C14663
- C14, C15, C16, C3: LCSC Part Number C23733 -> C1779
- C18, C19: LCSC Part Number C1548 -> C1644
- C22, C31, C37: LCSC Part Number C28323 -> C28323
- C32, C33: LCSC Part Number C15850 -> C28323
- C44, C45: LCSC Part Number C15850 -> (none); now left out of the parts list
- C46, C47, C48, C49: LCSC Part Number C15850 -> C14663
- D1, D2, D4, D5: LCSC Part Number C84256 -> C84256
- H1, H2, H3, H4, J10, J11, J13, J14, J15, J16, J17, J18, J19, J26, J27, J29, J30, J31, J5, J6, J7, J8, J9, R19, TP10, TP11, TP12, TP13, TP14, TP4, TP5, TP6, TP7, TP8, TP9: now left out of the parts list
- J12: LCSC Part Number (none) -> C22367949
- L1, L2, L3: LCSC Part Number (none) -> C42411119
- R1: LCSC Part Number C25105 -> C23140
- R10, R9: LCSC Part Number C25105 -> C23186
- R11, R12, R5: LCSC Part Number C11702 -> C21190
- R15, R23: LCSC Part Number C25792 -> C25803
- R16, R20, R21, R24, R28, R29: LCSC Part Number C25741 -> C25803
- R17, R4: LCSC Part Number C25076 -> C22775
- R18, R27: LCSC Part Number C25741 -> C25819
- R2, R3: LCSC Part Number C25092 -> C23140
- R22: LCSC Part Number C25792 -> C25819
- R25, R6: LCSC Part Number C25076 -> C23138
- R26: LCSC Part Number C25756 -> C22809
- R30: LCSC Part Number C25792 -> C23231
- R31: LCSC Part Number C25756 -> C22797
- R32, R33, R34, R35, R36, R37: LCSC Part Number C25744 -> C25804
- R7, R8: LCSC Part Number C25900 -> C23186
- SW1, SW2: LCSC Part Number (none) -> C115357
- U1: value W25Q128JVS -> W25Q128JVP; LCSC Part Number C97521 -> C190862
- U10: LCSC Part Number (none) -> SOT-23-8
- U11: LCSC Part Number (none) -> C23380830
- U15: LCSC Part Number (none) -> C2675635
- U2: LCSC Part Number (none) -> C42415655
- U4: LCSC Part Number (none) -> C22459454
- U6: LCSC Part Number (none) -> C699536
